Commit message: docs: update README with SLAM, troubleshooting, verified status
- README: added SLAM (2D Mapping) section with 5-terminal workflow,
  map save/reload commands
- README: added Troubleshooting section documenting the WSL2
  systemd-timesyncd -> gz-transport 7s stall diagnosis and fix
- README: added 'Latest Verified Status' section correcting the
  outdated 'Not started' notes
- .gitignore: exclude *.bak, frames_*.gv/pdf, map artifacts
- Add cmd_vel_watchdog.py (was untracked; fresh clone of the repo
  could not build because setup.py entry point referenced it)
- Accumulated changes from weeks 1-2 to urdf and world files

File: ros2_ws/src/patrol_robot/urdf/patrol_robot.urdf.xacro (robot description, xacro)
@@ -144,4 +144,48 @@
     <origin xyz="${-body_length / 2 + caster_radius} 0 ${-body_height / 2 - caster_radius}" rpy="0 0 0"/>
   </joint>
+  <!-- LiDAR sensoru: base_link uzerine sabitlenir -->
+  <link name="lidar_link">
+    <visual>
+      <geometry>
+        <cylinder radius="0.035" length="0.04"/>
+      </geometry>
+      <material name="lidar_black">
+        <color rgba="0.08 0.08 0.08 1.0"/>
+      </material>
+    </visual>
+    <inertial>
+      <mass value="0.1"/>
+      <inertia ixx="0.00005" ixy="0.0" ixz="0.0"
+               iyy="0.00005" iyz="0.0" izz="0.00005"/>
+    </inertial>
+  </link>
+  <joint name="lidar_joint" type="fixed">
+    <parent link="base_link"/>
+    <child link="lidar_link"/>
+    <origin xyz="0 0 0.08" rpy="0 0 0"/>
+  </joint>
+  <gazebo reference="lidar_link">
+    <sensor name="lidar_sensor" type="gpu_lidar">
+      <topic>/scan</topic>
+      <update_rate>10</update_rate>
+      <always_on>true</always_on>
+      <visualize>true</visualize>
+      <lidar>
+        <scan>
+          <horizontal>
+            <samples>360</samples>
+            <resolution>1</resolution>
+            <min_angle>-3.14159265</min_angle>
+            <max_angle>3.14159265</max_angle>
+          </horizontal>
+        </scan>
+        <range>
+          <min>0.12</min>
+          <max>8.0</max>
+          <resolution>0.01</resolution>
+        </range>
+      </lidar>
+    </sensor>
+  </gazebo>
   <!-- Gazebo diferansiyel surus eklentisi: /cmd_vel hiz komutunu tekerleklere cevirir -->
   <gazebo>
